File: JetCam.sch (KiCad schematic (older format))
At the start: 0 parts

Commit message: Add library and symbol for ADV7281A-M in a hierachical sheet named decoder
Parts:
- added J?: QTH-060-01-X-D-A, QTH-060-01-X-D-A, symbol QTH-060-01-X-D-A:QTH-060-01-X-D-A
Changed lines of the file:
@@
 EESchema Schematic File Version 4
+LIBS:JetCam-cache
 EELAYER 30 0
 EELAYER END
 $Descr A4 11693 8268
 encoding utf-8
-Sheet 1 1
+Sheet 1 2
 Title "Analogue to CSI camera board for the Jetson TX2 SDK"
 Date "2019-09-09"
@@
 Comment4 ""
 $EndDescr
+$Comp
+L QTH-060-01-X-D-A:QTH-060-01-X-D-A J?
+U 1 1 5D76E1D9
+P 5200 950
+F 0 "J?" H 5500 1217 50  0000 C CNN
+F 1 "QTH-060-01-X-D-A" H 5500 1126 50  0000 C CNN
+F 2 "QTH-060-01-X-D-A" H 5200 950 50  0001 L BNN
+F 3 "QTH-060-01-H-D-A" H 5200 950 50  0001 L BNN
+F 4 "https://www.digikey.com/product-detail/en/samtec-inc/QTH-060-01-H-D-A/SAM12792-ND/6695553?utm_source=snapeda&utm_medium=aggregator&utm_campaign=symbol" H 5200 950 50  0001 L BNN "Field4"
+F 5 "Samtec" H 5200 950 50  0001 L BNN "Field5"
+F 6 "None" H 5200 950 50  0001 L BNN "Field6"
+F 7 "SAM12792-ND" H 5200 950 50  0001 L BNN "Field7"
+F 8 "Connector Micro High Speed Terminal Strip HDR 120 POS 0.5mm Solder ST SMD Tube" H 5200 950 50  0001 L BNN "Field8"
+	1    5200 950
+	1    0    0    -1
+$EndComp
+$Sheet
+S 1700 1650 1300 2000
+U 5D773160
+F0 "decoder" 50
+F1 "decoder.sch" 50
+$EndSheet
 $EndSCHEMATC
